Commit message: update: 机械臂夹取demo

File: src/your_robot_gazebo/urdf/gazebo_moveit.urdf (robot description, URDF)
Before this commit: robot panda_primitive_pretty, 10 links, 9 joints
Links:
- added link finger_left, mass 0.08; collision box size=0.01 0.01 0.12; visual box size=0.01 0.01 0.12
- added link finger_right, mass 0.08; collision box size=0.01 0.01 0.12; visual box size=0.01 0.01 0.12
- added link gripper_base, mass 0.3; collision cylinder length=0.04 radius=0.03; visual cylinder length=0.04 radius=0.03
- added link tool0
- link ee_flange: mass None -> 0.2; geometry collision cylinder length=0.02 radius=0.05; visual cylinder length=0.02 radius=0.05
Joints:
- added joint finger_left_joint: type revolute, parent gripper_base, child finger_left, origin xyz=0 0.03 0, axis 1 0 0, limit lower=0 upper=0.7 effort=10 velocity=2.0
- added joint finger_right_joint: type revolute, parent gripper_base, child finger_right, origin xyz=0 -0.03 0, axis -1 0 0, limit lower=0 upper=0.7 effort=10 velocity=2.0
- added joint gripper_base_fixed: type fixed, parent ee_flange, child gripper_base, origin xyz=0 0 0.02
- added joint tool0_fixed: type fixed, parent gripper_base, child tool0, origin xyz=0 0 0.12
- joint ee_fixed: origin xyz=0 0 0.08 -> xyz=0 0 0.06

File: src/your_robot_gazebo/urdf/simplified.urdf (robot description, URDF)
Before this commit: robot panda_primitive_pretty, 10 links, 9 joints
Links:
- added link finger_left, mass 0.08; collision box size=0.01 0.01 0.12; visual box size=0.01 0.01 0.12
- added link finger_right, mass 0.08; collision box size=0.01 0.01 0.12; visual box size=0.01 0.01 0.12
- added link gripper_base, mass 0.3; collision cylinder length=0.04 radius=0.03; visual cylinder length=0.04 radius=0.03
- added link tool0
- link ee_flange: mass None -> 0.2; geometry collision cylinder length=0.02 radius=0.05; visual cylinder length=0.02 radius=0.05
Joints:
- added joint finger_left_joint: type revolute, parent gripper_base, child finger_left, origin xyz=0 0.03 0, axis 1 0 0, limit lower=0 upper=0.7 effort=10 velocity=2.0
- added joint finger_right_joint: type revolute, parent gripper_base, child finger_right, origin xyz=0 -0.03 0, axis -1 0 0, limit lower=0 upper=0.7 effort=10 velocity=2.0
- added joint gripper_base_fixed: type fixed, parent ee_flange, child gripper_base, origin xyz=0 0 0.02
- added joint tool0_fixed: type fixed, parent gripper_base, child tool0, origin xyz=0 0 0.12
- joint ee_fixed: origin xyz=0 0 0.08 -> xyz=0 0 0.06

File: src/your_robot_moveit/config/panda_primitive_pretty.ros2_control.xacro (robot description, xacro)
@@ -57,4 +57,18 @@
                 <state_interface name="velocity"/>
             </joint>
+            <joint name="finger_left_joint">
+                <command_interface name="position"/>
+                <state_interface name="position">
+                  <param name="initial_value">${initial_positions['finger_left_joint']}</param>
+                </state_interface>
+                <state_interface name="velocity"/>
+            </joint>
+            <joint name="finger_right_joint">
+                <command_interface name="position"/>
+                <state_interface name="position">
+                  <param name="initial_value">${initial_positions['finger_right_joint']}</param>
+                </state_interface>
+                <state_interface name="velocity"/>
+            </joint>
         </ros2_control>
     </xacro:macro>
